Commit message: Removed all Gazebo-related elements

File: description/face.xacro (robot description, xacro)
@@ -29,6 +29,3 @@
         </visual>
     </link>
-    <gazebo reference="face_link">
-        <material>Gazebo/Black</material>
-    </gazebo>
 </robot>

Commit message: Reconstructed Robi's RViz visuals and improved his behavior in narrow passages

File: description/face.xacro (robot description, xacro)
@@ -4,5 +4,5 @@
         <parent link="chassis"/>
         <child link="face_link"/>
-        <origin xyz="${chassis_length} 0 ${chassis_height/2}" rpy="0 0 0"/>
+        <origin xyz="0.125 0 ${chassis_height/2}" rpy="0 0 0"/>
     </joint>
     <link name="face_link">

File: description/lidar.xacro (robot description, xacro)
@@ -4,5 +4,5 @@
         <parent link="chassis"/>
         <child link="laser_frame"/>
-        <origin xyz="0.122 0 0.09" rpy="0 0 0"/>
+        <origin xyz="0.0 0 0.09" rpy="0 0 0"/>
     </joint>
     <link name="laser_frame">

File: description/robot.urdf.xacro (robot description, xacro)
@@ -11,5 +11,4 @@
     <xacro:include filename="lidar.xacro" />
     <xacro:include filename="camera.xacro" />
-    <!-- <xacro:include filename="depth_camera.xacro" /> -->
     <xacro:include filename="face.xacro" />
 </robot>

File: description/robot_core.xacro (robot description, xacro)
@@ -3,6 +3,6 @@
   <xacro:include filename="inertial_macros.xacro"/>
   <!-- Properties -->
-  <xacro:property name="chassis_length" value="0.2"/>
-  <xacro:property name="chassis_width" value="0.2"/>
+  <xacro:property name="chassis_length" value="0.25"/>
+  <xacro:property name="chassis_width" value="0.23"/>
   <xacro:property name="chassis_height" value="0.09"/>
   <xacro:property name="chassis_mass" value="1.0"/>
@@ -11,10 +11,6 @@
   <xacro:property name="wheel_mass" value="0.05"/>
   <xacro:property name="wheel_offset_x" value="0.11"/>
-  <xacro:property name="wheel_offset_y" value="0.11"/>
-  <xacro:property name="wheel_offset_z" value="0.01"/>
-  <xacro:property name="caster_wheel_radius" value="0.01"/>
-  <xacro:property name="caster_wheel_mass" value="0.01"/>
-  <xacro:property name="caster_wheel_offset_x" value="0.075"/>
-  <xacro:property name="caster_wheel_offset_z" value="${wheel_offset_z - wheel_radius + caster_wheel_radius}"/>
+  <xacro:property name="wheel_offset_y" value="0.115"/>
+  <xacro:property name="wheel_offset_z" value="0.0"/>
   <!-- Materials -->
   <material name="white"><color rgba="1 1 1 1" /></material>
@@ -39,5 +35,5 @@
   <link name="chassis">
     <visual>
-      <origin xyz="${chassis_length/2} 0 ${chassis_height/2}"/>
+      <origin xyz="0 0 ${chassis_height/2}"/>
       <geometry>
         <box size="${chassis_length} ${chassis_width} ${chassis_height}"/>
@@ -46,5 +42,5 @@
     </visual>
     <collision>
-      <origin xyz="${chassis_length/2} 0 ${chassis_height/2}"/>
+      <origin xyz="0 0 ${chassis_height/2}"/>
       <geometry>
         <box size="${chassis_length} ${chassis_width} ${chassis_height}"/>
@@ -52,61 +48,86 @@
     </collision>
     <xacro:inertial_box mass="0.5" x="${chassis_length}" y="${chassis_width}" z="${chassis_height}">
-      <origin xyz="${chassis_length/2} 0 ${chassis_height/2}" rpy="0 0 0"/>
+      <origin xyz="0 0 ${chassis_height/2}" rpy="0 0 0"/>
     </xacro:inertial_box>
   </link>
-  <!-- Wheels -->
-  <joint name="left_wheel_joint" type="continuous">
-    <parent link="chassis"/>
-    <child link="left_wheel"/>
-    <origin xyz="${wheel_offset_x} ${wheel_offset_y} 0" rpy="${pi/2} 0 0"/>
-    <axis xyz="0 0 1"/>
-  </joint>
-  <link name="left_wheel">
-    <visual>
-      <geometry><cylinder radius="${wheel_radius}" length="${wheel_thickness}"/></geometry>
-      <material name="blue"/>
-    </visual>
-    <collision>
-      <geometry><sphere radius="${wheel_radius}"/></geometry>
-    </collision>
-    <xacro:inertial_cylinder mass="${wheel_mass}" length="${wheel_thickness}" radius="${wheel_radius}">
-      <origin xyz="0 0 0" rpy="0 0 0"/>
-    </xacro:inertial_cylinder>
-  </link>
-  <joint name="right_wheel_joint" type="continuous">
-    <parent link="chassis"/>
-    <child link="right_wheel"/>
-    <origin xyz="${wheel_offset_x} ${-wheel_offset_y} 0" rpy="${pi/2} 0 0"/>
-    <axis xyz="0 0 1"/>
-  </joint>
-  <link name="right_wheel">
-    <visual>
-      <geometry><cylinder radius="${wheel_radius}" length="${wheel_thickness}"/></geometry>
-      <material name="blue"/>
-    </visual>
-    <collision>
-      <geometry><sphere radius="${wheel_radius}"/></geometry>
-    </collision>
-    <xacro:inertial_cylinder mass="${wheel_mass}" length="${wheel_thickness}" radius="${wheel_radius}">
-      <origin xyz="0 0 0" rpy="0 0 0"/>
-    </xacro:inertial_cylinder>
-  </link>
-  <!-- Caster Wheel -->
-  <joint name="caster_wheel_joint" type="fixed">
-    <parent link="chassis"/>
-    <child link="caster_wheel"/>
-    <origin xyz="${caster_wheel_offset_x} 0 ${caster_wheel_offset_z}"/>
-  </joint>
-  <link name="caster_wheel">
-    <visual>
-      <geometry><sphere radius="${caster_wheel_radius}"/></geometry>
-      <material name="white"/>
-    </visual>
-    <collision>
-      <geometry><sphere radius="${caster_wheel_radius}"/></geometry>
-    </collision>
-    <xacro:inertial_sphere mass="${caster_wheel_mass}" radius="${caster_wheel_radius}">
-      <origin xyz="0 0 0" rpy="0 0 0"/>
-    </xacro:inertial_sphere>
-  </link>
+<!--- Left Wheels - -->
+<joint name="left_front_wheel_joint" type="fixed">
+  <parent link="chassis"/>
+  <child link="left_front_wheel"/>
+  <origin xyz="0.08 ${wheel_offset_y} ${wheel_offset_z}" rpy="${pi/2} 0 0"/>
+</joint>
+<link name="left_front_wheel">
+  <visual>
+    <geometry>
+      <cylinder radius="${wheel_radius}" length="${wheel_thickness}"/>
+    </geometry>
+    <material name="blue"/>
+  </visual>
+</link>
+<joint name="left_mid_wheel_joint" type="fixed">
+  <parent link="chassis"/>
+  <child link="left_mid_wheel"/>
+  <origin xyz="0.0 ${wheel_offset_y} ${wheel_offset_z}" rpy="${pi/2} 0 0"/>
+</joint>
+<link name="left_mid_wheel">
+  <visual>
+    <geometry>
+      <cylinder radius="${wheel_radius}" length="${wheel_thickness}"/>
+    </geometry>
+    <material name="blue"/>
+  </visual>
+</link>
+<joint name="left_rear_wheel_joint" type="fixed">
+  <parent link="chassis"/>
+  <child link="left_rear_wheel"/>
+  <origin xyz="-0.08 ${wheel_offset_y} ${wheel_offset_z}" rpy="${pi/2} 0 0"/>
+</joint>
+<link name="left_rear_wheel">
+  <visual>
+    <geometry>
+      <cylinder radius="${wheel_radius}" length="${wheel_thickness}"/>
+    </geometry>
+    <material name="blue"/>
+  </visual>
+</link>
+<!-- - Right Wheels - -->
+<joint name="right_front_wheel_joint" type="fixed">
+  <parent link="chassis"/>
+  <child link="right_front_wheel"/>
+  <origin xyz="0.08 ${-wheel_offset_y} ${wheel_offset_z}" rpy="${pi/2} 0 0"/>
+</joint>
+<link name="right_front_wheel">
+  <visual>
+    <geometry>
+      <cylinder radius="${wheel_radius}" length="${wheel_thickness}"/>
+    </geometry>
+    <material name="blue"/>
+  </visual>
+</link>
+<joint name="right_mid_wheel_joint" type="fixed">
+  <parent link="chassis"/>
+  <child link="right_mid_wheel"/>
+  <origin xyz="0.0 ${-wheel_offset_y} ${wheel_offset_z}" rpy="${pi/2} 0 0"/>
+</joint>
+<link name="right_mid_wheel">
+  <visual>
+    <geometry>
+      <cylinder radius="${wheel_radius}" length="${wheel_thickness}"/>
+    </geometry>
+    <material name="blue"/>
+  </visual>
+</link>
+<joint name="right_rear_wheel_joint" type="fixed">
+  <parent link="chassis"/>
+  <child link="right_rear_wheel"/>
+  <origin xyz="-0.08 ${-wheel_offset_y} ${wheel_offset_z}" rpy="${pi/2} 0 0"/>
+</joint>
+<link name="right_rear_wheel">
+  <visual>
+    <geometry>
+      <cylinder radius="${wheel_radius}" length="${wheel_thickness}"/>
+    </geometry>
+    <material name="blue"/>
+  </visual>
+</link>
 </robot>
