Commit message: Removed all Gazebo-related elements

File: description/camera.xacro (robot description, xacro)
@@ -27,26 +27,3 @@
     </joint>
     <link name="camera_link_optical"></link>
-    <gazebo reference="camera_link">
-        <material>Gazebo/Black</material>
-        <sensor name="camera" type="camera">
-            <pose> 0 0 0 0 0 0 </pose>
-            <visualize>true</visualize>
-            <update_rate>10</update_rate>
-            <camera>
-                <horizontal_fov>1.089</horizontal_fov>
-                <image>
-                    <format>R8G8B8</format>
-                    <width>640</width>
-                    <height>480</height>
-                </image>
-                <clip>
-                    <near>0.05</near>
-                    <far>8.0</far>
-                </clip>
-            </camera>
-            <plugin name="camera_controller" filename="libgazebo_ros_camera.so">
-                <frame_name>camera_link_optical</frame_name>
-            </plugin>
-        </sensor>
-    </gazebo>
 </robot>

Commit message: Some Bug fixes

File: description/camera.xacro (robot description, xacro)
@@ -4,5 +4,5 @@
         <parent link="chassis"/>
         <child link="camera_link"/>
-        <origin xyz="0.276 0 0.181" rpy="0 0 0"/>
+        <origin xyz="0.24 0 0.09" rpy="0 0 0"/>
     </joint>
     <link name="camera_link">

File: description/lidar.xacro (robot description, xacro)
@@ -4,10 +4,10 @@
         <parent link="chassis"/>
         <child link="laser_frame"/>
-        <origin xyz="0.122 0 0.212" rpy="0 0 0"/>
+        <origin xyz="0.122 0 0.09" rpy="0 0 0"/>
     </joint>
     <link name="laser_frame">
         <visual>
             <geometry>
-                <cylinder radius="0.05" length="0.04"/>
+                <cylinder radius="0.035" length="0.04"/>
             </geometry>
             <material name="black"/>

File: description/robot_core.xacro (robot description, xacro)
@@ -2,13 +2,13 @@
 <robot xmlns:xacro="http://www.ros.org/wiki/xacro" >
     <xacro:include filename="inertial_macros.xacro"/>
-    <xacro:property name="chassis_length" value="0.335"/>
-    <xacro:property name="chassis_width" value="0.265"/>
-    <xacro:property name="chassis_height" value="0.138"/>
+    <xacro:property name="chassis_length" value="0.24"/>
+    <xacro:property name="chassis_width" value="0.23"/>
+    <xacro:property name="chassis_height" value="0.09"/>
     <xacro:property name="chassis_mass" value="1.0"/>
-    <xacro:property name="wheel_radius" value="0.033"/>
-    <xacro:property name="wheel_thickness" value="0.026"/>
+    <xacro:property name="wheel_radius" value="0.035"/>
+    <xacro:property name="wheel_thickness" value="0.04"/>
     <xacro:property name="wheel_mass" value="0.05"/>
-    <xacro:property name="wheel_offset_x" value="0.226"/>
-    <xacro:property name="wheel_offset_y" value="0.1485"/>
+    <xacro:property name="wheel_offset_x" value="0.11"/>
+    <xacro:property name="wheel_offset_y" value="0.11"/>
     <xacro:property name="wheel_offset_z" value="0.01"/>
     <xacro:property name="caster_wheel_radius" value="0.01"/>
@@ -71,5 +71,5 @@
         <parent link="chassis"/>
         <child link="left_wheel"/>
-        <origin xyz="${wheel_offset_x} ${wheel_offset_y} 0" rpy="-${pi/2} 0 0"/>
+        <origin xyz="${wheel_offset_x} ${wheel_offset_y} 0" rpy="${pi/2} 0 0"/>
         <axis xyz="0 0 1"/>
     </joint>

Commit message: Added a working setup enabling Robi’s real-world navigation

File: description/camera.xacro (robot description, xacro)
@@ -1,16 +1,26 @@
 <?xml version="1.0"?>
-<robot xmlns:xacro="http://www.ros.org/wiki/xacro">
+<robot name="camera_on_plate" xmlns:xacro="http://ros.org/wiki/xacro">
   <joint name="camera_joint" type="fixed">
-    <parent link="chassis"/>
+    <parent link="top_plate"/>
     <child link="camera_link"/>
-    <origin xyz="0.125 0 0.09" rpy="0 0 0"/>
+    <!-- Platte ist 0.17 m lang → Hälfte = 0.085 m.
+         Kamera-Tiefe = 0.01 m → Hälfte = 0.005 m.
+         Position x = 0.085 + 0.005 = 0.09 m -->
+    <origin xyz="0.09 0.0 0.0" rpy="0 0 0"/>
   </joint>
   <link name="camera_link">
     <visual>
       <geometry>
-        <box size="0.010 0.03 0.03"/>
+        <box size="0.010 0.030 0.030"/>
       </geometry>
-      <material name="black"/>
+      <material name="camera_black">
+        <color rgba="0 0 0 1"/>
+      </material>
     </visual>
+    <collision>
+      <geometry>
+        <box size="0.010 0.030 0.030"/>
+      </geometry>
+    </collision>
   </link>
   <joint name="camera_optical_joint" type="fixed">

File: description/face.xacro (robot description, xacro)
@@ -24,5 +24,5 @@
             <origin xyz="-0.011 0 -0.00" rpy="0 ${1.5} 0"/>
             <geometry>
-                <cylinder radius="0.05" length="0.02"/>
+                <cylinder radius="0.04" length="0.02"/>
             </geometry>
             <material name="red"/>

File: description/lidar.xacro (robot description, xacro)
@@ -1,49 +1,77 @@
 <?xml version="1.0"?>
-<xacro:macro name="lidar_setup" params="" xmlns:xacro="http://www.ros.org/wiki/xacro">
-  <joint name="servo_joint" type="continuous">
-    <parent link="chassis"/>
-    <child link="servo_link"/>
-    <origin xyz="0.0 0 0.09" rpy="0 0 0"/>
-    <axis xyz="0 1 0"/>
-  </joint>
-  <link name="servo_link">
-    <visual>
-      <origin xyz="0 0 0.025"/>
-      <geometry>
-        <cylinder radius="0.02" length="0.05"/>
-      </geometry>
-    </visual>
-  </link>
-  <joint name="laser_joint" type="fixed">
-    <parent link="servo_link"/>
-    <child link="laser_frame"/>
-    <origin xyz="0.0 0 0.05" rpy="0 0 0"/>
-  </joint>
-  <link name="laser_frame">
-    <visual>
-      <geometry>
-        <cylinder radius="0.035" length="0.04"/>
-      </geometry>
-      <material name="black"/>
-    </visual>
-    <visual>
-      <origin xyz="0 0 -0.05"/>
-      <geometry>
-        <cylinder radius="0.01" length="0.1"/>
-      </geometry>
-      <material name="black"/>
-    </visual>
-    <collision>
-      <geometry>
-        <cylinder radius="0.05" length="0.04"/>
-      </geometry>
-    </collision>
-    <inertial>
-      <mass value="0.1"/>
-      <origin xyz="0 0 0" rpy="0 0 0"/>
-      <inertia ixx="0.01" ixy="0.0" ixz="0.0"
-               iyy="0.01" iyz="0.0"
-               izz="0.01"/>
-    </inertial>
-  </link>
-</xacro:macro>
+<robot name="lidar_lib" xmlns:xacro="http://www.ros.org/wiki/xacro">
+  <xacro:macro name="lidar_setup" params="parent:=top_plate
+                                          servo_link:=servo_link
+                                          laser_frame:=laser_frame">
+    <material name="lidar_black"><color rgba="0.05 0.05 0.05 1.0"/></material>
+    <material name="lidar_gray"><color rgba="0.5 0.5 0.5 1.0"/></material>
+    <material name="lidar_blue"><color rgba="0.2 0.5 1.0 1.0"/></material>
+    <joint name="lidar_mount_joint" type="fixed">
+      <parent link="${parent}"/>
+      <child link="lidar_mount"/>
+      <origin xyz="0 0 0.02" rpy="0 0 0"/>
+    </joint>
+    <link name="lidar_mount">
+      <visual>
+        <geometry><box size="0.05 0.05 0.04"/></geometry>
+        <material name="lidar_gray"/>
+      </visual>
+      <collision>
+        <geometry><box size="0.05 0.05 0.04"/></geometry>
+      </collision>
+      <inertial>
+        <mass value="0.15"/>
+        <origin xyz="0 0 0" rpy="0 0 0"/>
+        <inertia ixx="0.0003" ixy="0" ixz="0" iyy="0.0003" iyz="0" izz="0.0003"/>
+      </inertial>
+    </link>
+    <joint name="servo_joint" type="continuous">
+      <parent link="lidar_mount"/>
+      <child link="${servo_link}"/>
+      <origin xyz="0 0 0.02" rpy="0 0 0"/>
+      <axis xyz="0 1 0"/>
+    </joint>
+    <link name="${servo_link}">
+      <visual>
+        <origin xyz="0 0 0.0175" rpy="0 0 0"/>
+        <geometry><cylinder radius="0.008" length="0.035"/></geometry>
+        <material name="lidar_gray"/>
+      </visual>
+      <collision>
+        <origin xyz="0 0 0.0175" rpy="0 0 0"/>
+        <geometry><cylinder radius="0.008" length="0.035"/></geometry>
+      </collision>
+      <inertial>
+        <mass value="0.05"/>
+        <origin xyz="0 0 0" rpy="0 0 0"/>
+        <inertia ixx="0.0001" ixy="0" ixz="0" iyy="0.0001" iyz="0" izz="0.0001"/>
+      </inertial>
+    </link>
+    <joint name="laser_joint" type="fixed">
+      <parent link="${servo_link}"/>
+      <child link="${laser_frame}"/>
+      <origin xyz="0 0 0.04" rpy="0 0 0"/>
+    </joint>
+    <link name="${laser_frame}">
+      <visual>
+        <origin xyz="0 0 0.02" rpy="0 0 0"/>
+        <geometry><cylinder radius="0.04" length="0.05"/></geometry>
+        <material name="lidar_black"/>
+      </visual>
+      <collision>
+        <origin xyz="0 0 0.02" rpy="0 0 0"/>
+        <geometry><cylinder radius="0.04" length="0.05"/></geometry>
+      </collision>
+      <visual>
+        <origin xyz="0 0 0" rpy="0 0 0"/>
+        <geometry><cylinder radius="0.041" length="0.0015"/></geometry>
+        <material name="lidar_blue"/>
+      </visual>
+      <inertial>
+        <mass value="0.25"/>
+        <origin xyz="0 0 0.02" rpy="0 0 0"/>
+        <inertia ixx="0.002" ixy="0" ixz="0" iyy="0.002" iyz="0" izz="0.002"/>
+      </inertial>
+    </link>
+  </xacro:macro>
+</robot>

File: description/robot.urdf.xacro (robot description, xacro)
@@ -10,4 +10,5 @@
     </xacro:if>
     <xacro:include filename="lidar.xacro" />
+    <xacro:lidar_setup parent="top_plate" servo_link="servo_link" laser_frame="laser_frame" />
     <xacro:include filename="camera.xacro" />
     <xacro:include filename="face.xacro" />

File: description/robot_core.xacro (robot description, xacro)
@@ -131,3 +131,111 @@
   </visual>
 </link>
+  <xacro:property name="standoff_height" value="0.07"/>
+  <xacro:property name="standoff_radius" value="0.005"/>
+  <xacro:property name="plate_length" value="0.17"/>
+  <xacro:property name="plate_width"  value="0.18"/>
+  <xacro:property name="plate_thickness" value="0.003"/>
+  <xacro:property name="standoff_inset_x" value="0.02"/>
+  <xacro:property name="standoff_inset_y" value="0.02"/>
+  <xacro:property name="metal_rgba" value="0.7 0.7 0.7 1"/>
+  <material name="metal_gray"><color rgba="${metal_rgba}"/></material>
+  <xacro:property name="plate_center_x" value="0.01"/>
+  <xacro:property name="plate_center_y" value="0.0"/>
+  <xacro:property name="plate_center_z" value="${chassis_height + standoff_height + plate_thickness/2}"/>
+  <xacro:property name="sx" value="${(plate_length/2) - standoff_inset_x}"/>
+  <xacro:property name="sy" value="${(plate_width/2)  - standoff_inset_y}"/>
+  <xacro:property name="standoff_center_z" value="${chassis_height + standoff_height/2}"/>
+  <joint name="standoff_fl_joint" type="fixed">
+    <parent link="chassis"/>
+    <child link="standoff_fl"/>
+    <origin xyz="${plate_center_x + sx} ${plate_center_y + sy} ${standoff_center_z}" rpy="0 0 0"/>
+  </joint>
+  <link name="standoff_fl">
+    <visual>
+      <geometry>
+        <cylinder radius="${standoff_radius}" length="${standoff_height}"/>
+      </geometry>
+      <material name="metal_gray"/>
+    </visual>
+    <collision>
+      <geometry>
+        <cylinder radius="${standoff_radius}" length="${standoff_height}"/>
+      </geometry>
+    </collision>
+  </link>
+  <joint name="standoff_fr_joint" type="fixed">
+    <parent link="chassis"/>
+    <child link="standoff_fr"/>
+    <origin xyz="${plate_center_x + sx} ${plate_center_y - sy} ${standoff_center_z}" rpy="0 0 0"/>
+  </joint>
+  <link name="standoff_fr">
+    <visual>
+      <geometry>
+        <cylinder radius="${standoff_radius}" length="${standoff_height}"/>
+      </geometry>
+      <material name="metal_gray"/>
+    </visual>
+    <collision>
+      <geometry>
+        <cylinder radius="${standoff_radius}" length="${standoff_height}"/>
+      </geometry>
+    </collision>
+  </link>
+  <joint name="standoff_rl_joint" type="fixed">
+    <parent link="chassis"/>
+    <child link="standoff_rl"/>
+    <origin xyz="${plate_center_x - sx} ${plate_center_y + sy} ${standoff_center_z}" rpy="0 0 0"/>
+  </joint>
+  <link name="standoff_rl">
+    <visual>
+      <geometry>
+        <cylinder radius="${standoff_radius}" length="${standoff_height}"/>
+      </geometry>
+      <material name="metal_gray"/>
+    </visual>
+    <collision>
+      <geometry>
+        <cylinder radius="${standoff_radius}" length="${standoff_height}"/>
+      </geometry>
+    </collision>
+  </link>
+  <joint name="standoff_rr_joint" type="fixed">
+    <parent link="chassis"/>
+    <child link="standoff_rr"/>
+    <origin xyz="${plate_center_x - sx} ${plate_center_y - sy} ${standoff_center_z}" rpy="0 0 0"/>
+  </joint>
+  <link name="standoff_rr">
+    <visual>
+      <geometry>
+        <cylinder radius="${standoff_radius}" length="${standoff_height}"/>
+      </geometry>
+      <material name="metal_gray"/>
+    </visual>
+    <collision>
+      <geometry>
+        <cylinder radius="${standoff_radius}" length="${standoff_height}"/>
+      </geometry>
+    </collision>
+  </link>
+  <joint name="top_plate_joint" type="fixed">
+    <parent link="chassis"/>
+    <child link="top_plate"/>
+    <origin xyz="${plate_center_x} ${plate_center_y} ${plate_center_z}" rpy="0 0 0"/>
+  </joint>
+  <link name="top_plate">
+    <visual>
+      <geometry>
+        <box size="${plate_length} ${plate_width} ${plate_thickness}"/>
+      </geometry>
+      <material name="metal_gray"/>
+    </visual>
+    <collision>
+      <geometry>
+        <box size="${plate_length} ${plate_width} ${plate_thickness}"/>
+      </geometry>
+    </collision>
+    <xacro:inertial_box mass="0.3" x="${plate_length}" y="${plate_width}" z="${plate_thickness}">
+      <origin xyz="0 0 0" rpy="0 0 0"/>
+    </xacro:inertial_box>
+  </link>
 </robot>
