Commit message: Added real-time timestamp adjustment for LaserScan messages and increased transform tolerance to improve TF stability

File: description/robot.urdf.xacro (robot description, xacro)
@@ -1,5 +1,5 @@
 <?xml version="1.0"?>
 <robot xmlns:xacro="http://www.ros.org/wiki/xacro"  name="robot">
-    <xacro:arg name="use_ros2_control" default="true"/>
+    <xacro:arg name="use_ros2_control" default="false"/>
     <xacro:arg name="sim_mode" default="false"/>
     <xacro:arg name="esp_ip" default="192.168.1.100"/>

File: description/robot_core.xacro (robot description, xacro)
@@ -1,137 +1,112 @@
 <?xml version="1.0"?>
-<robot xmlns:xacro="http://www.ros.org/wiki/xacro" >
-    <xacro:include filename="inertial_macros.xacro"/>
-    <xacro:property name="chassis_length" value="0.2"/>
-    <xacro:property name="chassis_width" value="0.2"/>
-    <xacro:property name="chassis_height" value="0.09"/>
-    <xacro:property name="chassis_mass" value="1.0"/>
-    <xacro:property name="wheel_radius" value="0.035"/>
-    <xacro:property name="wheel_thickness" value="0.04"/>
-    <xacro:property name="wheel_mass" value="0.05"/>
-    <xacro:property name="wheel_offset_x" value="0.11"/>
-    <xacro:property name="wheel_offset_y" value="0.11"/>
-    <xacro:property name="wheel_offset_z" value="0.01"/>
-    <xacro:property name="caster_wheel_radius" value="0.01"/>
-    <xacro:property name="caster_wheel_mass" value="0.01"/>
-    <xacro:property name="caster_wheel_offset_x" value="0.075"/>
-    <xacro:property name="caster_wheel_offset_z" value="${wheel_offset_z - wheel_radius + caster_wheel_radius}"/>
-    <material name="white">
-        <color rgba="1 1 1 1" />
-    </material>
-    <material name="orange">
-        <color rgba="1 0.3 0.1 1"/>
-    </material>
-    <material name="blue">
-        <color rgba="0.2 0.2 1 1"/>
-    </material>
-    <material name="black">
-        <color rgba="0 0 0 1"/>
-    </material>
-    <material name="red">
-        <color rgba="1 0 0 1"/>
-    </material>
-    <!-- BASE LINK -->
-    <link name="base_link">
-    </link>
-    <!-- CHASSIS LINK -->
-    <joint name="base_footprint_joint" type="fixed">
-        <parent link="base_link"/>
-        <child link="base_footprint"/>
-        <origin xyz="0 0 0" rpy="0 0 0"/>
-    </joint>
-    <!-- BASE LINK -->
-    <link name="base_footprint">
-    </link>
-    <!-- CHASSIS LINK -->
-    <joint name="chassis_joint" type="fixed">
-        <parent link="base_link"/>
-        <child link="chassis"/>
-        <origin xyz="0 0 0"/>
-    </joint>
-    <link name="chassis">
-        <visual>
-            <origin xyz="${chassis_length/2} 0 ${chassis_height/2}"/>
-            <geometry>
-                <box size="${chassis_length} ${chassis_width} ${chassis_height}"/>
-            </geometry>
-            <material name="orange"/>
-        </visual>
-        <collision>
-            <origin xyz="${chassis_length/2} 0 ${chassis_height/2}"/>
-            <geometry>
-                <box size="${chassis_length} ${chassis_width} ${chassis_height}"/>
-            </geometry>
-        </collision>
-        <xacro:inertial_box mass="0.5" x="${chassis_length}" y="${chassis_width}" z="${chassis_height}">
-            <origin xyz="${chassis_length/2} 0 ${chassis_height/2}" rpy="0 0 0"/>
-        </xacro:inertial_box>
-    </link>
-    <!-- LEFT WHEEL LINK -->
-    <joint name="left_wheel_joint" type="continuous">
-        <parent link="chassis"/>
-        <child link="left_wheel"/>
-        <origin xyz="${wheel_offset_x} ${wheel_offset_y} 0" rpy="${pi/2} 0 0"/>
-        <axis xyz="0 0 1"/>
-    </joint>
-    <link name="left_wheel">
-        <visual>
-            <geometry>
-                <cylinder radius="${wheel_radius}" length="${wheel_thickness}"/>
-            </geometry>
-            <material name="blue"/>
-        </visual>
-        <collision>
-            <geometry>
-                <sphere radius="${wheel_radius}"/>
-            </geometry>
-        </collision>
-        <xacro:inertial_cylinder mass="${wheel_mass}" length="${wheel_thickness}" radius="${wheel_radius}">
-            <origin xyz="0 0 0" rpy="0 0 0"/>
-        </xacro:inertial_cylinder>
-    </link>
-    <!-- RIGHT WHEEL LINK -->
-    <joint name="right_wheel_joint" type="continuous">
-        <parent link="chassis"/>
-        <child link="right_wheel"/>
-        <origin xyz="${wheel_offset_x} ${-wheel_offset_y} 0" rpy="${pi/2}  0 0"/>
-        <axis xyz="0 0 1"/>
-    </joint>
-    <link name="right_wheel">
-        <visual>
-            <geometry>
-                <cylinder radius="${wheel_radius}" length="${wheel_thickness}"/>
-            </geometry>
-            <material name="blue"/>
-        </visual>
-        <collision>
-            <geometry>
-                <sphere radius="${wheel_radius}"/>
-            </geometry>
-        </collision>
-        <xacro:inertial_cylinder mass="${wheel_mass}" length="${wheel_thickness}" radius="${wheel_radius}">
-            <origin xyz="0 0 0" rpy="0 0 0"/>
-        </xacro:inertial_cylinder>
-    </link>
-    <!-- CASTER WHEEL LINK -->
-    <joint name="caster_wheel_joint" type="fixed">
-        <parent link="chassis"/>
-        <child link="caster_wheel"/>
-        <origin xyz="${caster_wheel_offset_x} 0 ${caster_wheel_offset_z}"/>
-    </joint>
-    <link name="caster_wheel">
-        <visual>
-            <geometry>
-                <sphere radius="${caster_wheel_radius}"/>
-            </geometry>
-            <material name="white"/>
-        </visual>
-        <collision>
-            <geometry>
-                <sphere radius="${caster_wheel_radius}"/>
-            </geometry>
-        </collision>
-        <xacro:inertial_sphere mass="${caster_wheel_mass}" radius="${caster_wheel_radius}">
-            <origin xyz="0 0 0" rpy="0 0 0"/>
-        </xacro:inertial_sphere>
-    </link>
+<robot xmlns:xacro="http://www.ros.org/wiki/xacro">
+  <xacro:include filename="inertial_macros.xacro"/>
+  <!-- Properties -->
+  <xacro:property name="chassis_length" value="0.2"/>
+  <xacro:property name="chassis_width" value="0.2"/>
+  <xacro:property name="chassis_height" value="0.09"/>
+  <xacro:property name="chassis_mass" value="1.0"/>
+  <xacro:property name="wheel_radius" value="0.035"/>
+  <xacro:property name="wheel_thickness" value="0.04"/>
+  <xacro:property name="wheel_mass" value="0.05"/>
+  <xacro:property name="wheel_offset_x" value="0.11"/>
+  <xacro:property name="wheel_offset_y" value="0.11"/>
+  <xacro:property name="wheel_offset_z" value="0.01"/>
+  <xacro:property name="caster_wheel_radius" value="0.01"/>
+  <xacro:property name="caster_wheel_mass" value="0.01"/>
+  <xacro:property name="caster_wheel_offset_x" value="0.075"/>
+  <xacro:property name="caster_wheel_offset_z" value="${wheel_offset_z - wheel_radius + caster_wheel_radius}"/>
+  <!-- Materials -->
+  <material name="white"><color rgba="1 1 1 1" /></material>
+  <material name="orange"><color rgba="1 0.3 0.1 1"/></material>
+  <material name="blue"><color rgba="0.2 0.2 1 1"/></material>
+  <material name="black"><color rgba="0 0 0 1"/></material>
+  <material name="red"><color rgba="1 0 0 1"/></material>
+  <!-- Base -->
+  <link name="base_link"/>
+  <joint name="base_footprint_joint" type="fixed">
+    <parent link="base_link"/>
+    <child link="base_footprint"/>
+    <origin xyz="0 0 0" rpy="0 0 0"/>
+  </joint>
+  <link name="base_footprint"/>
+  <!-- Chassis -->
+  <joint name="chassis_joint" type="fixed">
+    <parent link="base_link"/>
+    <child link="chassis"/>
+    <origin xyz="0 0 0"/>
+  </joint>
+  <link name="chassis">
+    <visual>
+      <origin xyz="${chassis_length/2} 0 ${chassis_height/2}"/>
+      <geometry>
+        <box size="${chassis_length} ${chassis_width} ${chassis_height}"/>
+      </geometry>
+      <material name="orange"/>
+    </visual>
+    <collision>
+      <origin xyz="${chassis_length/2} 0 ${chassis_height/2}"/>
+      <geometry>
+        <box size="${chassis_length} ${chassis_width} ${chassis_height}"/>
+      </geometry>
+    </collision>
+    <xacro:inertial_box mass="0.5" x="${chassis_length}" y="${chassis_width}" z="${chassis_height}">
+      <origin xyz="${chassis_length/2} 0 ${chassis_height/2}" rpy="0 0 0"/>
+    </xacro:inertial_box>
+  </link>
+  <!-- Wheels -->
+  <joint name="left_wheel_joint" type="continuous">
+    <parent link="chassis"/>
+    <child link="left_wheel"/>
+    <origin xyz="${wheel_offset_x} ${wheel_offset_y} 0" rpy="${pi/2} 0 0"/>
+    <axis xyz="0 0 1"/>
+  </joint>
+  <link name="left_wheel">
+    <visual>
+      <geometry><cylinder radius="${wheel_radius}" length="${wheel_thickness}"/></geometry>
+      <material name="blue"/>
+    </visual>
+    <collision>
+      <geometry><sphere radius="${wheel_radius}"/></geometry>
+    </collision>
+    <xacro:inertial_cylinder mass="${wheel_mass}" length="${wheel_thickness}" radius="${wheel_radius}">
+      <origin xyz="0 0 0" rpy="0 0 0"/>
+    </xacro:inertial_cylinder>
+  </link>
+  <joint name="right_wheel_joint" type="continuous">
+    <parent link="chassis"/>
+    <child link="right_wheel"/>
+    <origin xyz="${wheel_offset_x} ${-wheel_offset_y} 0" rpy="${pi/2} 0 0"/>
+    <axis xyz="0 0 1"/>
+  </joint>
+  <link name="right_wheel">
+    <visual>
+      <geometry><cylinder radius="${wheel_radius}" length="${wheel_thickness}"/></geometry>
+      <material name="blue"/>
+    </visual>
+    <collision>
+      <geometry><sphere radius="${wheel_radius}"/></geometry>
+    </collision>
+    <xacro:inertial_cylinder mass="${wheel_mass}" length="${wheel_thickness}" radius="${wheel_radius}">
+      <origin xyz="0 0 0" rpy="0 0 0"/>
+    </xacro:inertial_cylinder>
+  </link>
+  <!-- Caster Wheel -->
+  <joint name="caster_wheel_joint" type="fixed">
+    <parent link="chassis"/>
+    <child link="caster_wheel"/>
+    <origin xyz="${caster_wheel_offset_x} 0 ${caster_wheel_offset_z}"/>
+  </joint>
+  <link name="caster_wheel">
+    <visual>
+      <geometry><sphere radius="${caster_wheel_radius}"/></geometry>
+      <material name="white"/>
+    </visual>
+    <collision>
+      <geometry><sphere radius="${caster_wheel_radius}"/></geometry>
+    </collision>
+    <xacro:inertial_sphere mass="${caster_wheel_mass}" radius="${caster_wheel_radius}">
+      <origin xyz="0 0 0" rpy="0 0 0"/>
+    </xacro:inertial_sphere>
+  </link>
 </robot>

Commit message: rovi can now drive around with his new wheels

File: description/robot.urdf.xacro (robot description, xacro)
@@ -7,5 +7,5 @@
     <xacro:if value="$(arg use_ros2_control)">
         <xacro:include filename="ros2_control.xacro" />
-        <xacro:ros2_control_config esp_ip="$(arg esp_ip)" />
+        <xacro:ros2_control_config />
     </xacro:if>
     <xacro:include filename="lidar.xacro" />

File: description/robot_core.xacro (robot description, xacro)
@@ -19,6 +19,7 @@
   <material name="black"><color rgba="0 0 0 1"/></material>
   <material name="red"><color rgba="1 0 0 1"/></material>
-  <!-- Base -->
+  <!-- BASE LINK -->
   <link name="base_link"/>
+  <!-- BASE_FOOTPRINT LINK -->
   <joint name="base_footprint_joint" type="fixed">
     <parent link="base_link"/>
@@ -27,5 +28,5 @@
   </joint>
   <link name="base_footprint"/>
-  <!-- Chassis -->
+  <!-- CHASSIS LINK -->
   <joint name="chassis_joint" type="fixed">
     <parent link="base_link"/>
@@ -51,62 +52,96 @@
     </xacro:inertial_box>
   </link>
-<!--- Left Wheels - -->
-<joint name="left_front_wheel_joint" type="continuous">
-  <axis xyz="0 1 0"/>
-  <parent link="chassis"/>
-  <child link="left_front_wheel"/>
-  <origin xyz="0.08 ${wheel_offset_y} ${wheel_offset_z}" rpy="${pi/2} 0 0"/>
-</joint>
-<link name="left_front_wheel">
-  <visual>
-    <geometry>
-      <cylinder radius="${wheel_radius}" length="${wheel_thickness}"/>
-    </geometry>
-    <material name="blue"/>
-  </visual>
-</link>
-<joint name="left_rear_wheel_joint" type="continuous">
-  <axis xyz="0 1 0"/>
-  <parent link="chassis"/>
-  <child link="left_rear_wheel"/>
-  <origin xyz="-0.08 ${wheel_offset_y} ${wheel_offset_z}" rpy="${pi/2} 0 0"/>
-</joint>
-<link name="left_rear_wheel">
-  <visual>
-    <geometry>
-      <cylinder radius="${wheel_radius}" length="${wheel_thickness}"/>
-    </geometry>
-    <material name="blue"/>
-  </visual>
-</link>
-<!-- - Right Wheels - -->
-<joint name="right_front_wheel_joint" type="continuous">
-  <axis xyz="0 1 0"/>
-  <parent link="chassis"/>
-  <child link="right_front_wheel"/>
-  <origin xyz="0.08 ${-wheel_offset_y} ${wheel_offset_z}" rpy="${pi/2} 0 0"/>
-</joint>
-<link name="right_front_wheel">
-  <visual>
-    <geometry>
-      <cylinder radius="${wheel_radius}" length="${wheel_thickness}"/>
-    </geometry>
-    <material name="blue"/>
-  </visual>
-</link>
-<joint name="right_rear_wheel_joint" type="continuous">
-  <axis xyz="0 1 0"/>
-  <parent link="chassis"/>
-  <child link="right_rear_wheel"/>
-  <origin xyz="-0.08 ${-wheel_offset_y} ${wheel_offset_z}" rpy="${pi/2} 0 0"/>
-</joint>
-<link name="right_rear_wheel">
-  <visual>
-    <geometry>
-      <cylinder radius="${wheel_radius}" length="${wheel_thickness}"/>
-    </geometry>
-    <material name="blue"/>
-  </visual>
-</link>
+  <!-- LEFT FRONT WHEEL -->
+  <joint name="left_front_wheel_joint" type="continuous">
+    <axis xyz="0 1 0"/>
+    <parent link="chassis"/>
+    <child link="left_front_wheel"/>
+    <origin xyz="0.08 ${wheel_offset_y} ${wheel_offset_z}" rpy="${pi/2} 0 0"/>
+  </joint>
+  <link name="left_front_wheel">
+    <visual>
+      <geometry>
+        <cylinder radius="${wheel_radius}" length="${wheel_thickness}"/>
+      </geometry>
+      <material name="blue"/>
+    </visual>
+    <collision>
+      <geometry>
+        <sphere radius="${wheel_radius}"/>
+      </geometry>
+    </collision>
+    <xacro:inertial_cylinder mass="${wheel_mass}" length="${wheel_thickness}" radius="${wheel_radius}">
+      <origin xyz="0 0 0" rpy="0 0 0"/>
+    </xacro:inertial_cylinder>
+  </link>
+  <!-- LEFT REAR WHEEL -->
+  <joint name="left_rear_wheel_joint" type="continuous">
+    <axis xyz="0 1 0"/>
+    <parent link="chassis"/>
+    <child link="left_rear_wheel"/>
+    <origin xyz="-0.08 ${wheel_offset_y} ${wheel_offset_z}" rpy="${pi/2} 0 0"/>
+  </joint>
+  <link name="left_rear_wheel">
+    <visual>
+      <geometry>
+        <cylinder radius="${wheel_radius}" length="${wheel_thickness}"/>
+      </geometry>
+      <material name="blue"/>
+    </visual>
+    <collision>
+      <geometry>
+        <sphere radius="${wheel_radius}"/>
+      </geometry>
+    </collision>
+    <xacro:inertial_cylinder mass="${wheel_mass}" length="${wheel_thickness}" radius="${wheel_radius}">
+      <origin xyz="0 0 0" rpy="0 0 0"/>
+    </xacro:inertial_cylinder>
+  </link>
+  <!-- RIGHT FRONT WHEEL -->
+  <joint name="right_front_wheel_joint" type="continuous">
+    <axis xyz="0 1 0"/>
+    <parent link="chassis"/>
+    <child link="right_front_wheel"/>
+    <origin xyz="0.08 ${-wheel_offset_y} ${wheel_offset_z}" rpy="${pi/2} 0 0"/>
+  </joint>
+  <link name="right_front_wheel">
+    <visual>
+      <geometry>
+        <cylinder radius="${wheel_radius}" length="${wheel_thickness}"/>
+      </geometry>
+      <material name="blue"/>
+    </visual>
+    <collision>
+      <geometry>
+        <sphere radius="${wheel_radius}"/>
+      </geometry>
+    </collision>
+    <xacro:inertial_cylinder mass="${wheel_mass}" length="${wheel_thickness}" radius="${wheel_radius}">
+      <origin xyz="0 0 0" rpy="0 0 0"/>
+    </xacro:inertial_cylinder>
+  </link>
+  <!-- RIGHT REAR WHEEL -->
+  <joint name="right_rear_wheel_joint" type="continuous">
+    <axis xyz="0 1 0"/>
+    <parent link="chassis"/>
+    <child link="right_rear_wheel"/>
+    <origin xyz="-0.08 ${-wheel_offset_y} ${wheel_offset_z}" rpy="${pi/2} 0 0"/>
+  </joint>
+  <link name="right_rear_wheel">
+    <visual>
+      <geometry>
+        <cylinder radius="${wheel_radius}" length="${wheel_thickness}"/>
+      </geometry>
+      <material name="blue"/>
+    </visual>
+    <collision>
+      <geometry>
+        <sphere radius="${wheel_radius}"/>
+      </geometry>
+    </collision>
+    <xacro:inertial_cylinder mass="${wheel_mass}" length="${wheel_thickness}" radius="${wheel_radius}">
+      <origin xyz="0 0 0" rpy="0 0 0"/>
+    </xacro:inertial_cylinder>
+  </link>
   <xacro:property name="standoff_height" value="0.07"/>
   <xacro:property name="standoff_radius" value="0.005"/>

File: description/ros2_control.xacro (robot description, xacro)
@@ -1,14 +1,17 @@
 <?xml version="1.0"?>
 <robot xmlns:xacro="http://www.ros.org/wiki/xacro">
-    <xacro:arg name="esp_ip" default="192.168.1.100"/>
-    <xacro:macro name="ros2_control_config" params="esp_ip">
-        <ros2_control name="RealRobot" type="system">
+    <xacro:macro name="ros2_control_config">
+        <ros2_control name="DiffDriveArduino" type="system">
             <hardware>
-                <plugin>mock_components/GenericSystem</plugin>
-                <param name="esp_ip">http://$(arg esp_ip)</param> <!-- ESP IP-Adresse -->
-                <param name="baud_rate">115200</param> <!-- Angepasste Baudrate -->
+                <plugin>diffdrive_arduino/DiffDriveArduino</plugin>
+                <param name="left_wheel_name">left_wheel_joint</param>
+                <param name="right_wheel_name">right_wheel_joint</param>
+                <param name="loop_rate">30</param>
+                <param name="device">/dev/ttyACM0</param>
+                <param name="baud_rate">57600</param>
                 <param name="timeout">1000</param>
+                <param name="enc_counts_per_rev">3436</param>
             </hardware>
-            <joint name="left_front_wheel_joint">
+            <joint name="left_wheel_joint">
                 <command_interface name="velocity">
                     <param name="min">-10</param>
@@ -18,21 +21,5 @@
                 <state_interface name="position"/>
             </joint>
-            <joint name="left_rear_wheel_joint">
-                <command_interface name="velocity">
-                    <param name="min">-10</param>
-                    <param name="max">10</param>
-                </command_interface>
-                <state_interface name="velocity"/>
-                <state_interface name="position"/>
-            </joint>
-            <joint name="right_front_wheel_joint">
-                <command_interface name="velocity">
-                    <param name="min">-10</param>
-                    <param name="max">10</param>
-                </command_interface>
-                <state_interface name="velocity"/>
-                <state_interface name="position"/>
-            </joint>
-            <joint name="right_rear_wheel_joint">
+            <joint name="right_wheel_joint">
                 <command_interface name="velocity">
                     <param name="min">-10</param>
