Commit message: Changed a few things to simplify the reproduction

File: description/robot_core.xacro (robot description, xacro)
@@ -2,6 +2,6 @@
 <robot xmlns:xacro="http://www.ros.org/wiki/xacro" >
     <xacro:include filename="inertial_macros.xacro"/>
-    <xacro:property name="chassis_length" value="0.24"/>
-    <xacro:property name="chassis_width" value="0.23"/>
+    <xacro:property name="chassis_length" value="0.2"/>
+    <xacro:property name="chassis_width" value="0.2"/>
     <xacro:property name="chassis_height" value="0.09"/>
     <xacro:property name="chassis_mass" value="1.0"/>

Commit message: fixing motor issues

File: description/robot_core.xacro (robot description, xacro)
@@ -54,5 +54,5 @@
   <!-- LEFT FRONT WHEEL -->
   <joint name="left_front_wheel_joint" type="continuous">
-    <axis xyz="0 1 0"/>
+    <axis xyz="0 0 1"/>
     <parent link="chassis"/>
     <child link="left_front_wheel"/>
@@ -77,5 +77,5 @@
   <!-- LEFT REAR WHEEL -->
   <joint name="left_rear_wheel_joint" type="continuous">
-    <axis xyz="0 1 0"/>
+    <axis xyz="0 0 1"/>
     <parent link="chassis"/>
     <child link="left_rear_wheel"/>
@@ -100,5 +100,5 @@
   <!-- RIGHT FRONT WHEEL -->
   <joint name="right_front_wheel_joint" type="continuous">
-    <axis xyz="0 1 0"/>
+    <axis xyz="0 0 1"/>
     <parent link="chassis"/>
     <child link="right_front_wheel"/>
@@ -123,5 +123,5 @@
   <!-- RIGHT REAR WHEEL -->
   <joint name="right_rear_wheel_joint" type="continuous">
-    <axis xyz="0 1 0"/>
+    <axis xyz="0 0 1"/>
     <parent link="chassis"/>
     <child link="right_rear_wheel"/>
