Commit message: Removed all Gazebo-related elements

File: description/lidar.xacro (robot description, xacro)
@@ -29,31 +29,3 @@
         </xacro:inertial_cylinder>
     </link>
-    <gazebo reference="laser_frame">
-        <material>Gazebo/Black</material>
-        <sensor name="laser" type="ray">
-            <pose> 0 0 0 0 0 0 </pose>
-            <visualize>false</visualize>
-            <update_rate>10</update_rate>
-            <ray>
-                <scan>
-                    <horizontal>
-                        <samples>360</samples>
-                        <min_angle>-3.14</min_angle>
-                        <max_angle>3.14</max_angle>
-                    </horizontal>
-                </scan>
-                <range>
-                    <min>0.3</min>
-                    <max>12</max>
-                </range>
-            </ray>
-            <plugin name="laser_controller" filename="libgazebo_ros_ray_sensor.so">
-                <ros>
-                    <argument>~/out:=scan</argument>
-                </ros>
-                <output_type>sensor_msgs/LaserScan</output_type>
-                <frame_name>laser_frame</frame_name>
-            </plugin>
-        </sensor>
-    </gazebo>
 </robot>

Commit message: Add working 3D Lidar version

File: description/lidar.xacro (robot description, xacro)
@@ -1,31 +1,49 @@
 <?xml version="1.0"?>
-<robot xmlns:xacro="http://www.ros.org/wiki/xacro" >
-    <joint name="laser_joint" type="fixed">
-        <parent link="chassis"/>
-        <child link="laser_frame"/>
-        <origin xyz="0.0 0 0.09" rpy="0 0 0"/>
-    </joint>
-    <link name="laser_frame">
-        <visual>
-            <geometry>
-                <cylinder radius="0.035" length="0.04"/>
-            </geometry>
-            <material name="black"/>
-        </visual>
-        <visual>
-            <origin xyz="0 0 -0.05"/>
-            <geometry>
-                <cylinder radius="0.01" length="0.1"/>
-            </geometry>
-            <material name="black"/>
-        </visual>
-        <collision>
-            <geometry>
-                <cylinder radius="0.05" length="0.04"/>
-            </geometry>
-        </collision>
-        <xacro:inertial_cylinder mass="0.1" length="0.04" radius="0.05">
-            <origin xyz="0 0 0" rpy="0 0 0"/>
-        </xacro:inertial_cylinder>
-    </link>
-</robot>
+<xacro:macro name="lidar_setup" params="" xmlns:xacro="http://www.ros.org/wiki/xacro">
+  <joint name="servo_joint" type="continuous">
+    <parent link="chassis"/>
+    <child link="servo_link"/>
+    <origin xyz="0.0 0 0.09" rpy="0 0 0"/>
+    <axis xyz="0 1 0"/>
+  </joint>
+  <link name="servo_link">
+    <visual>
+      <origin xyz="0 0 0.025"/>
+      <geometry>
+        <cylinder radius="0.02" length="0.05"/>
+      </geometry>
+    </visual>
+  </link>
+  <joint name="laser_joint" type="fixed">
+    <parent link="servo_link"/>
+    <child link="laser_frame"/>
+    <origin xyz="0.0 0 0.05" rpy="0 0 0"/>
+  </joint>
+  <link name="laser_frame">
+    <visual>
+      <geometry>
+        <cylinder radius="0.035" length="0.04"/>
+      </geometry>
+      <material name="black"/>
+    </visual>
+    <visual>
+      <origin xyz="0 0 -0.05"/>
+      <geometry>
+        <cylinder radius="0.01" length="0.1"/>
+      </geometry>
+      <material name="black"/>
+    </visual>
+    <collision>
+      <geometry>
+        <cylinder radius="0.05" length="0.04"/>
+      </geometry>
+    </collision>
+    <inertial>
+      <mass value="0.1"/>
+      <origin xyz="0 0 0" rpy="0 0 0"/>
+      <inertia ixx="0.01" ixy="0.0" ixz="0.0"
+               iyy="0.01" iyz="0.0"
+               izz="0.01"/>
+    </inertial>
+  </link>
+</xacro:macro>

Commit message: Bug fixing

File: description/lidar.xacro (robot description, xacro)
@@ -30,5 +30,5 @@
       <child link="${servo_link}"/>
       <origin xyz="0 0 0.02" rpy="0 0 0"/>
-      <axis xyz="0 1 0"/>
+      <axis xyz="0 -1 0"/>
     </joint>
     <link name="${servo_link}">

Commit message: Adding pololu motors

File: description/lidar.xacro (robot description, xacro)
@@ -1,77 +1,30 @@
 <?xml version="1.0"?>
-<robot name="lidar_lib" xmlns:xacro="http://www.ros.org/wiki/xacro">
-  <xacro:macro name="lidar_setup" params="parent:=top_plate
-                                          servo_link:=servo_link
-                                          laser_frame:=laser_frame">
-    <material name="lidar_black"><color rgba="0.05 0.05 0.05 1.0"/></material>
-    <material name="lidar_gray"><color rgba="0.5 0.5 0.5 1.0"/></material>
-    <material name="lidar_blue"><color rgba="0.2 0.5 1.0 1.0"/></material>
-    <joint name="lidar_mount_joint" type="fixed">
-      <parent link="${parent}"/>
-      <child link="lidar_mount"/>
-      <origin xyz="0 0 0.02" rpy="0 0 0"/>
+<robot xmlns:xacro="http://www.ros.org/wiki/xacro" >
+    <joint name="laser_joint" type="fixed">
+        <parent link="chassis"/>
+        <child link="laser_frame"/>
+        <origin xyz="0.0 0 0.09" rpy="0 0 0"/>
     </joint>
-    <link name="lidar_mount">
-      <visual>
-        <geometry><box size="0.05 0.05 0.04"/></geometry>
-        <material name="lidar_gray"/>
-      </visual>
-      <collision>
-        <geometry><box size="0.05 0.05 0.04"/></geometry>
-      </collision>
-      <inertial>
-        <mass value="0.15"/>
-        <origin xyz="0 0 0" rpy="0 0 0"/>
-        <inertia ixx="0.0003" ixy="0" ixz="0" iyy="0.0003" iyz="0" izz="0.0003"/>
-      </inertial>
+    <link name="laser_frame">
+        <visual>
+            <geometry>
+                <cylinder radius="0.035" length="0.04"/>
+            </geometry>
+            <material name="black"/>
+        </visual>
+        <visual>
+            <geometry>
+                <cylinder radius="0.01" length="0.1"/>
+            </geometry>
+            <material name="black"/>
+        </visual>
+        <collision>
+            <geometry>
+                <cylinder radius="0.05" length="0.04"/>
+            </geometry>
+        </collision>
+        <xacro:inertial_cylinder mass="0.1" length="0.04" radius="0.05">
+            <origin xyz="0 0 0" rpy="0 0 0"/>
+        </xacro:inertial_cylinder>
     </link>
-    <joint name="servo_joint" type="continuous">
-      <parent link="lidar_mount"/>
-      <child link="${servo_link}"/>
-      <origin xyz="0 0 0.02" rpy="0 0 0"/>
-      <axis xyz="0 -1 0"/>
-    </joint>
-    <link name="${servo_link}">
-      <visual>
-        <origin xyz="0 0 0.0175" rpy="0 0 0"/>
-        <geometry><cylinder radius="0.008" length="0.035"/></geometry>
-        <material name="lidar_gray"/>
-      </visual>
-      <collision>
-        <origin xyz="0 0 0.0175" rpy="0 0 0"/>
-        <geometry><cylinder radius="0.008" length="0.035"/></geometry>
-      </collision>
-      <inertial>
-        <mass value="0.05"/>
-        <origin xyz="0 0 0" rpy="0 0 0"/>
-        <inertia ixx="0.0001" ixy="0" ixz="0" iyy="0.0001" iyz="0" izz="0.0001"/>
-      </inertial>
-    </link>
-    <joint name="laser_joint" type="fixed">
-      <parent link="${servo_link}"/>
-      <child link="${laser_frame}"/>
-      <origin xyz="0 0 0.04" rpy="0 0 0"/>
-    </joint>
-    <link name="${laser_frame}">
-      <visual>
-        <origin xyz="0 0 0.02" rpy="0 0 0"/>
-        <geometry><cylinder radius="0.04" length="0.05"/></geometry>
-        <material name="lidar_black"/>
-      </visual>
-      <collision>
-        <origin xyz="0 0 0.02" rpy="0 0 0"/>
-        <geometry><cylinder radius="0.04" length="0.05"/></geometry>
-      </collision>
-      <visual>
-        <origin xyz="0 0 0" rpy="0 0 0"/>
-        <geometry><cylinder radius="0.041" length="0.0015"/></geometry>
-        <material name="lidar_blue"/>
-      </visual>
-      <inertial>
-        <mass value="0.25"/>
-        <origin xyz="0 0 0.02" rpy="0 0 0"/>
-        <inertia ixx="0.002" ixy="0" ixz="0" iyy="0.002" iyz="0" izz="0.002"/>
-      </inertial>
-    </link>
-  </xacro:macro>
 </robot>

File: description/robot.urdf_3d.xacro (robot description, xacro)
@@ -10,4 +10,5 @@
     </xacro:if>
     <xacro:include filename="lidar.xacro" />
+    <xacro:lidar_setup parent="top_plate" servo_link="servo_link" laser_frame="laser_frame" />
     <xacro:include filename="camera.xacro" />
     <xacro:include filename="face.xacro" />

File: description/robot_core.xacro (robot description, xacro)
@@ -52,5 +52,6 @@
   </link>
 <!--- Left Wheels - -->
-<joint name="left_front_wheel_joint" type="fixed">
+<joint name="left_front_wheel_joint" type="continuous">
+  <axis xyz="0 1 0"/>
   <parent link="chassis"/>
   <child link="left_front_wheel"/>
@@ -65,18 +66,6 @@
   </visual>
 </link>
-<joint name="left_mid_wheel_joint" type="fixed">
-  <parent link="chassis"/>
-  <child link="left_mid_wheel"/>
-  <origin xyz="0.0 ${wheel_offset_y} ${wheel_offset_z}" rpy="${pi/2} 0 0"/>
-</joint>
-<link name="left_mid_wheel">
-  <visual>
-    <geometry>
-      <cylinder radius="${wheel_radius}" length="${wheel_thickness}"/>
-    </geometry>
-    <material name="blue"/>
-  </visual>
-</link>
-<joint name="left_rear_wheel_joint" type="fixed">
+<joint name="left_rear_wheel_joint" type="continuous">
+  <axis xyz="0 1 0"/>
   <parent link="chassis"/>
   <child link="left_rear_wheel"/>
@@ -92,5 +81,6 @@
 </link>
 <!-- - Right Wheels - -->
-<joint name="right_front_wheel_joint" type="fixed">
+<joint name="right_front_wheel_joint" type="continuous">
+  <axis xyz="0 1 0"/>
   <parent link="chassis"/>
   <child link="right_front_wheel"/>
@@ -105,18 +95,6 @@
   </visual>
 </link>
-<joint name="right_mid_wheel_joint" type="fixed">
-  <parent link="chassis"/>
-  <child link="right_mid_wheel"/>
-  <origin xyz="0.0 ${-wheel_offset_y} ${wheel_offset_z}" rpy="${pi/2} 0 0"/>
-</joint>
-<link name="right_mid_wheel">
-  <visual>
-    <geometry>
-      <cylinder radius="${wheel_radius}" length="${wheel_thickness}"/>
-    </geometry>
-    <material name="blue"/>
-  </visual>
-</link>
-<joint name="right_rear_wheel_joint" type="fixed">
+<joint name="right_rear_wheel_joint" type="continuous">
+  <axis xyz="0 1 0"/>
   <parent link="chassis"/>
   <child link="right_rear_wheel"/>

File: description/ros2_control.xacro (robot description, xacro)
@@ -10,5 +10,5 @@
                 <param name="timeout">1000</param>
             </hardware>
-            <joint name="left_wheel_joint">
+            <joint name="left_front_wheel_joint">
                 <command_interface name="velocity">
                     <param name="min">-10</param>
@@ -18,5 +18,21 @@
                 <state_interface name="position"/>
             </joint>
-            <joint name="right_wheel_joint">
+            <joint name="left_rear_wheel_joint">
+                <command_interface name="velocity">
+                    <param name="min">-10</param>
+                    <param name="max">10</param>
+                </command_interface>
+                <state_interface name="velocity"/>
+                <state_interface name="position"/>
+            </joint>
+            <joint name="right_front_wheel_joint">
+                <command_interface name="velocity">
+                    <param name="min">-10</param>
+                    <param name="max">10</param>
+                </command_interface>
+                <state_interface name="velocity"/>
+                <state_interface name="position"/>
+            </joint>
+            <joint name="right_rear_wheel_joint">
                 <command_interface name="velocity">
                     <param name="min">-10</param>

Commit message: 3d und 2D mapping

File: description/lidar.xacro (robot description, xacro)
@@ -1,30 +1,77 @@
 <?xml version="1.0"?>
-<robot xmlns:xacro="http://www.ros.org/wiki/xacro" >
+<robot name="lidar_lib" xmlns:xacro="http://www.ros.org/wiki/xacro">
+  <xacro:macro name="lidar_setup" params="parent:=top_plate
+                                          servo_link:=servo_link
+                                          laser_frame:=laser_frame">
+    <material name="lidar_black"><color rgba="0.05 0.05 0.05 1.0"/></material>
+    <material name="lidar_gray"><color rgba="0.5 0.5 0.5 1.0"/></material>
+    <material name="lidar_blue"><color rgba="0.2 0.5 1.0 1.0"/></material>
+    <joint name="lidar_mount_joint" type="fixed">
+      <parent link="${parent}"/>
+      <child link="lidar_mount"/>
+      <origin xyz="0 0 0.02" rpy="0 0 0"/>
+    </joint>
+    <link name="lidar_mount">
+      <visual>
+        <geometry><box size="0.05 0.05 0.04"/></geometry>
+        <material name="lidar_gray"/>
+      </visual>
+      <collision>
+        <geometry><box size="0.05 0.05 0.04"/></geometry>
+      </collision>
+      <inertial>
+        <mass value="0.15"/>
+        <origin xyz="0 0 0" rpy="0 0 0"/>
+        <inertia ixx="0.0003" ixy="0" ixz="0" iyy="0.0003" iyz="0" izz="0.0003"/>
+      </inertial>
+    </link>
+    <joint name="servo_joint" type="continuous">
+      <parent link="lidar_mount"/>
+      <child link="${servo_link}"/>
+      <origin xyz="0 0 0.02" rpy="0 0 0"/>
+      <axis xyz="0 -1 0"/>
+    </joint>
+    <link name="${servo_link}">
+      <visual>
+        <origin xyz="0 0 0.0175" rpy="0 0 0"/>
+        <geometry><cylinder radius="0.008" length="0.035"/></geometry>
+        <material name="lidar_gray"/>
+      </visual>
+      <collision>
+        <origin xyz="0 0 0.0175" rpy="0 0 0"/>
+        <geometry><cylinder radius="0.008" length="0.035"/></geometry>
+      </collision>
+      <inertial>
+        <mass value="0.05"/>
+        <origin xyz="0 0 0" rpy="0 0 0"/>
+        <inertia ixx="0.0001" ixy="0" ixz="0" iyy="0.0001" iyz="0" izz="0.0001"/>
+      </inertial>
+    </link>
     <joint name="laser_joint" type="fixed">
-        <parent link="chassis"/>
-        <child link="laser_frame"/>
-        <origin xyz="0.0 0 0.09" rpy="0 0 0"/>
+      <parent link="${servo_link}"/>
+      <child link="${laser_frame}"/>
+      <origin xyz="0 0 0.04" rpy="0 0 0"/>
     </joint>
-    <link name="laser_frame">
-        <visual>
-            <geometry>
-                <cylinder radius="0.035" length="0.04"/>
-            </geometry>
-            <material name="black"/>
-        </visual>
-        <visual>
-            <geometry>
-                <cylinder radius="0.01" length="0.1"/>
-            </geometry>
-            <material name="black"/>
-        </visual>
-        <collision>
-            <geometry>
-                <cylinder radius="0.05" length="0.04"/>
-            </geometry>
-        </collision>
-        <xacro:inertial_cylinder mass="0.1" length="0.04" radius="0.05">
-            <origin xyz="0 0 0" rpy="0 0 0"/>
-        </xacro:inertial_cylinder>
+    <link name="${laser_frame}">
+      <visual>
+        <origin xyz="0 0 0.02" rpy="0 0 0"/>
+        <geometry><cylinder radius="0.04" length="0.05"/></geometry>
+        <material name="lidar_black"/>
+      </visual>
+      <collision>
+        <origin xyz="0 0 0.02" rpy="0 0 0"/>
+        <geometry><cylinder radius="0.04" length="0.05"/></geometry>
+      </collision>
+      <visual>
+        <origin xyz="0 0 0" rpy="0 0 0"/>
+        <geometry><cylinder radius="0.041" length="0.0015"/></geometry>
+        <material name="lidar_blue"/>
+      </visual>
+      <inertial>
+        <mass value="0.25"/>
+        <origin xyz="0 0 0.02" rpy="0 0 0"/>
+        <inertia ixx="0.002" ixy="0" ixz="0" iyy="0.002" iyz="0" izz="0.002"/>
+      </inertial>
     </link>
+  </xacro:macro>
 </robot>

File: description/robot.urdf.xacro (robot description, xacro)
@@ -7,7 +7,8 @@
     <xacro:if value="$(arg use_ros2_control)">
         <xacro:include filename="ros2_control.xacro" />
-        <xacro:ros2_control_config />
+        <xacro:ros2_control_config esp_ip="$(arg esp_ip)" />
     </xacro:if>
-    <xacro:include filename="lidar.xacro" />
+    <xacro:include filename="lidar_3d.xacro" />
+    <xacro:lidar_setup parent="top_plate" servo_link="servo_link" laser_frame="laser_frame" />
     <xacro:include filename="camera.xacro" />
     <xacro:include filename="face.xacro" />

File: description/robot.urdf_3d.xacro (robot description, xacro)
@@ -9,5 +9,5 @@
         <xacro:ros2_control_config esp_ip="$(arg esp_ip)" />
     </xacro:if>
-    <xacro:include filename="lidar.xacro" />
+    <xacro:include filename="lidar_3d.xacro" />
     <xacro:lidar_setup parent="top_plate" servo_link="servo_link" laser_frame="laser_frame" />
     <xacro:include filename="camera.xacro" />

File: description/robot_core.xacro (robot description, xacro)
@@ -19,7 +19,6 @@
   <material name="black"><color rgba="0 0 0 1"/></material>
   <material name="red"><color rgba="1 0 0 1"/></material>
-  <!-- BASE LINK -->
+  <!-- Base -->
   <link name="base_link"/>
-  <!-- BASE_FOOTPRINT LINK -->
   <joint name="base_footprint_joint" type="fixed">
     <parent link="base_link"/>
@@ -28,5 +27,5 @@
   </joint>
   <link name="base_footprint"/>
-  <!-- CHASSIS LINK -->
+  <!-- Chassis -->
   <joint name="chassis_joint" type="fixed">
     <parent link="base_link"/>

File: description/ros2_control.xacro (robot description, xacro)
@@ -1,15 +1,12 @@
 <?xml version="1.0"?>
 <robot xmlns:xacro="http://www.ros.org/wiki/xacro">
-    <xacro:macro name="ros2_control_config">
-        <ros2_control name="DiffDriveArduino" type="system">
+    <xacro:arg name="esp_ip" default="192.168.1.100"/>
+    <xacro:macro name="ros2_control_config" params="esp_ip">
+        <ros2_control name="RealRobot" type="system">
             <hardware>
-                <plugin>diffdrive_arduino/DiffDriveArduino</plugin>
-                <param name="left_wheel_name">left_wheel_joint</param>
-                <param name="right_wheel_name">right_wheel_joint</param>
-                <param name="loop_rate">30</param>
-                <param name="device">/dev/ttyACM0</param>
-                <param name="baud_rate">57600</param>
+                <plugin>mock_components/GenericSystem</plugin>
+                <param name="esp_ip">http://$(arg esp_ip)</param> <!-- ESP IP-Adresse -->
+                <param name="baud_rate">115200</param> <!-- Angepasste Baudrate -->
                 <param name="timeout">1000</param>
-                <param name="enc_counts_per_rev">3436</param>
             </hardware>
             <joint name="left_wheel_joint">
